File: BusMonitor.sch (KiCad schematic (older format))
At the start: 6 parts, among them U10 LCD_I2C_Generic, U8 MCP23017_SP, U9 MCP23017_SP

Commit message: Tie IO expander resets to Arduino reset.
Connections:
- wire segments 52 -> 59
- no-connect marks 38 -> 35
Changed lines of the file:
@@
 NoConn ~ 8050 3600
 NoConn ~ 8050 3700
-NoConn ~ 8050 3900
 NoConn ~ 7150 3100
 NoConn ~ 7150 3200
@@
 NoConn ~ 5750 3600
 NoConn ~ 5750 3700
-NoConn ~ 5750 3900
 Wire Wire Line
 	5750 4400 5700 4400
@@
 Wire Wire Line
 	6450 5000 6450 4950
-NoConn ~ 4850 3200
 NoConn ~ 4850 3300
 NoConn ~ 4450 2800
@@
 Wire Bus Line
 	3550 3500 3550 5600
+Connection ~ 3550 5600
+Wire Bus Line
+	3550 5600 7500 5600
+Wire Wire Line
+	4850 3200 5350 3200
+Wire Wire Line
+	5350 3200 5350 3900
+Wire Wire Line
+	5350 3900 5750 3900
+Wire Wire Line
+	5350 3200 5350 2250
+Wire Wire Line
+	5350 2250 7650 2250
+Wire Wire Line
+	7650 2250 7650 3900
+Wire Wire Line
+	7650 3900 8050 3900
 Wire Bus Line
 	7450 4000 7450 5500
 Wire Bus Line
 	9800 3100 9800 5400
-Connection ~ 3550 5600
-Wire Bus Line
-	3550 5600 7500 5600
+Connection ~ 5350 3200
 $EndSCHEMATC

Commit message: Add sync connection.
Connections:
- net labels added: SYNC
- wire segments 59 -> 60
- no-connect marks 35 -> 34
Changed lines of the file:
@@
-$EndComp
-$Comp
-L Interface_Expansion:MCP23017_SP U8
-U 1 1 60F32103
-P 6450 3800
-F 0 "U8" H 6000 4750 50  0000 C CNN
-F 1 "MCP23017_SP" H 6750 4750 50  0000 C CNN
-F 2 "Package_DIP:DIP-28_W7.62mm" H 6650 2800 50  0001 L CNN
-F 3 "http://ww1.microchip.com/downloads/en/DeviceDoc/20001952C.pdf" H 6650 2700 50  0001 L CNN
-	1    6450 3800
-	1    0    0    -1
 $EndComp
 $Comp
@@
 NoConn ~ 8050 3600
 NoConn ~ 8050 3700
-NoConn ~ 7150 3100
 NoConn ~ 7150 3200
 NoConn ~ 7150 3300
@@
 Wire Bus Line
 	1200 5600 3550 5600
-Wire Bus Line
-	7500 3100 7500 5600
 $Comp
 L Device:R R3
@@
 Wire Wire Line
 	7650 3900 8050 3900
+Connection ~ 5350 3200
+$Comp
+L Interface_Expansion:MCP23017_SP U8
+U 1 1 60F32103
+P 6450 3800
+F 0 "U8" H 6000 4750 50  0000 C CNN
+F 1 "MCP23017_SP" H 6750 4750 50  0000 C CNN
+F 2 "Package_DIP:DIP-28_W7.62mm" H 6650 2800 50  0001 L CNN
+F 3 "http://ww1.microchip.com/downloads/en/DeviceDoc/20001952C.pdf" H 6650 2700 50  0001 L CNN
+	1    6450 3800
+	1    0    0    -1
+$EndComp
+Wire Wire Line
+	7150 3100 7400 3100
+Entry Wire Line
+	7400 3100 7500 3200
+Text Label 7200 3100 0    50   ~ 0
+SYNC
+Wire Bus Line
+	7500 3100 7500 5600
 Wire Bus Line
 	7450 4000 7450 5500
 Wire Bus Line
 	9800 3100 9800 5400
-Connection ~ 5350 3200
 $EndSCHEMATC

Commit message: Add footprints to schematic.
Parts:
- R3, R4: footprint (none) -> Resistor_THT:R_Axial_DIN0207_L6.3mm_D2.5mm_P7.62mm_Horizontal
- U10: footprint (none) -> Connector_PinHeader_2.54mm:PinHeader_1x04_P2.54mm_Vertical
Changed lines of the file:
@@
 Text Label 9500 4600 0    50   ~ 0
 A7
-Wire Wire Line
-	9450 3000 9700 3000
 Entry Wire Line
 	9700 3000 9800 3100
@@
 F 0 "R3" V 3000 2400 50  0000 C CNN
 F 1 "4.7k" V 3050 2250 50  0000 C CNN
-F 2 "" V 2980 2250 50  0001 C CNN
+F 2 "Resistor_THT:R_Axial_DIN0207_L6.3mm_D2.5mm_P7.62mm_Horizontal" V 2980 2250 50  0001 C CNN
 F 3 "~" H 3050 2250 50  0001 C CNN
 	1    3050 2250
@@
 F 0 "R4" V 3000 2550 50  0000 C CNN
 F 1 "4.7k" V 3050 2400 50  0000 C CNN
-F 2 "" V 2980 2400 50  0001 C CNN
+F 2 "Resistor_THT:R_Axial_DIN0207_L6.3mm_D2.5mm_P7.62mm_Horizontal" V 2980 2400 50  0001 C CNN
 F 3 "~" H 3050 2400 50  0001 C CNN
 	1    3050 2400
@@
 F 0 "U10" H 2830 3996 50  0000 L CNN
 F 1 "LCD_I2C_Generic" H 2830 3905 50  0000 L CNN
-F 2 "" H 2400 3350 50  0001 C CNN
+F 2 "Connector_PinHeader_2.54mm:PinHeader_1x04_P2.54mm_Vertical" H 2400 3350 50  0001 C CNN
 F 3 "" H 2400 3450 50  0001 C CNN
 	1    2400 3950
@@
 Text Label 7200 3100 0    50   ~ 0
 SYNC
+Wire Wire Line
+	9450 3000 9700 3000
 Wire Bus Line
 	7500 3100 7500 5600
