File: MWC 6502 v1.0.sch (KiCad schematic (older format))
At the start: 19 parts, among them SW1 PWR_RES, U1 74HC00, U2 74HC00, U3 DS1233, U4 74HC00, U5 LM7805_TO220, U6 74HC00, U7 LM555xN

Commit message: Add footprints to schematic.
Parts:
- C1, C3, C6: footprint (none) -> Capacitor_THT:CP_Radial_D5.0mm_P2.50mm
- C2, C5: footprint (none) -> Capacitor_THT:C_Disc_D7.5mm_W5.0mm_P7.50mm
- C4, C7, C8, C9: footprint (none) -> Capacitor_THT:C_Disc_D4.3mm_W1.9mm_P5.00mm
- R1, R2: footprint (none) -> Resistor_THT:R_Axial_DIN0207_L6.3mm_D2.5mm_P7.62mm_Horizontal
- SW1: footprint (none) -> Button_Switch_THT:SW_PUSH_6mm
- U1: footprint (none) -> Package_DIP:DIP-16_W7.62mm_Socket
- U2: value 74HC00 -> 65C02S; footprint (none) -> Package_DIP:DIP-40_W15.24mm_Socket
- U3: footprint (none) -> Package_TO_SOT_THT:TO-92_Inline_Wide
- U4: value 74HC00 -> 62256; footprint (none) -> Package_DIP:DIP-28_W15.24mm_Socket
- U6: value 74HC00 -> 28C256; footprint (none) -> Socket:DIP_Socket-28_W11.9_W12.7_W15.24_W17.78_W18.5_3M_228-1277-00-0602J
Changed lines of the file:
@@
 P 1600 2400
 F 0 "U2" H 1350 3800 50  0000 C CNN
-F 1 "74HC00" H 1800 3800 50  0000 C CNN
-F 2 "" V 1600 2400 50  0001 C CNN
-F 3 "http://www.ti.com/lit/gpn/sn74hc00" H 1600 2800 50  0001 C CNN
+F 1 "65C02S" H 1800 3800 50  0000 C CNN
+F 2 "Package_DIP:DIP-40_W15.24mm_Socket" V 1600 2400 50  0001 C CNN
+F 3 "" H 1600 2800 50  0001 C CNN
 	1    1600 2400
 	1    0    0    -1
@@
 P 3500 2050
 F 0 "U4" H 3250 3100 50  0000 C CNN
-F 1 "74HC00" H 3700 3100 50  0000 C CNN
-F 2 "" H 3500 2050 50  0001 C CNN
-F 3 "http://www.ti.com/lit/gpn/sn74hc00" H 3500 2050 50  0001 C CNN
+F 1 "62256" H 3700 3100 50  0000 C CNN
+F 2 "Package_DIP:DIP-28_W15.24mm_Socket" H 3500 2050 50  0001 C CNN
+F 3 "" H 3500 2050 50  0001 C CNN
 	1    3500 2050
 	1    0    0    -1
@@
 F 0 "U1" H 1550 6975 50  0000 C CNN
 F 1 "74HC00" H 1550 6884 50  0000 C CNN
-F 2 "" H 1550 6650 50  0001 C CNN
+F 2 "Package_DIP:DIP-16_W7.62mm_Socket" H 1550 6650 50  0001 C CNN
 F 3 "http://www.ti.com/lit/gpn/sn74hc00" H 1550 6650 50  0001 C CNN
 	2    1550 6650
@@
 P 5350 2050
 F 0 "U6" H 5100 3100 50  0000 C CNN
-F 1 "74HC00" H 5550 3100 50  0000 C CNN
-F 2 "" H 5350 2050 50  0001 C CNN
-F 3 "http://www.ti.com/lit/gpn/sn74hc00" H 5350 2050 50  0001 C CNN
+F 1 "28C256" H 5550 3100 50  0000 C CNN
+F 2 "Socket:DIP_Socket-28_W11.9_W12.7_W15.24_W17.78_W18.5_3M_228-1277-00-0602J" H 5350 2050 50  0001 C CNN
+F 3 "" H 5350 2050 50  0001 C CNN
 	1    5350 2050
 	1    0    0    -1
@@
 F 0 "U1" H 1550 6425 50  0000 C CNN
 F 1 "74HC00" H 1550 6334 50  0000 C CNN
-F 2 "" H 1550 6100 50  0001 C CNN
+F 2 "Package_DIP:DIP-16_W7.62mm_Socket" H 1550 6100 50  0001 C CNN
 F 3 "http://www.ti.com/lit/gpn/sn74hc00" H 1550 6100 50  0001 C CNN
 	4    1550 6100
@@
 F 0 "U1" H 1550 5875 50  0000 C CNN
 F 1 "74HC00" H 1550 5784 50  0000 C CNN
-F 2 "" H 1550 5550 50  0001 C CNN
+F 2 "Package_DIP:DIP-16_W7.62mm_Socket" H 1550 5550 50  0001 C CNN
 F 3 "http://www.ti.com/lit/gpn/sn74hc00" H 1550 5550 50  0001 C CNN
 	3    1550 5550
@@
 F 0 "U1" H 1550 7525 50  0000 C CNN
 F 1 "74HC00" H 1550 7434 50  0000 C CNN
-F 2 "" H 1550 7200 50  0001 C CNN
+F 2 "Package_DIP:DIP-16_W7.62mm_Socket" H 1550 7200 50  0001 C CNN
 F 3 "http://www.ti.com/lit/gpn/sn74hc00" H 1550 7200 50  0001 C CNN
 	1    1550 7200
@@
 F 0 "U1" H 4550 7500 50  0000 C CNN
 F 1 "74HC00" H 4850 7500 50  0000 C CNN
-F 2 "" H 4700 7150 50  0001 C CNN
+F 2 "Package_DIP:DIP-16_W7.62mm_Socket" H 4700 7150 50  0001 C CNN
 F 3 "http://www.ti.com/lit/gpn/sn74hc00" H 4700 7150 50  0001 C CNN
 	5    4700 7150
@@
 F 0 "U3" H 2620 5396 50  0000 R CNN
 F 1 "DS1233" H 2620 5305 50  0000 R CNN
-F 2 "" H 2450 5500 50  0001 C CNN
+F 2 "Package_TO_SOT_THT:TO-92_Inline_Wide" H 2450 5500 50  0001 C CNN
 F 3 "" H 2550 5600 50  0001 C CNN
 	1    2850 5350
@@
 F 0 "C2" H 3415 5596 50  0000 L CNN
 F 1 ".01uF" H 3415 5505 50  0000 L CNN
-F 2 "" H 3338 5400 50  0001 C CNN
+F 2 "Capacitor_THT:C_Disc_D7.5mm_W5.0mm_P7.50mm" H 3338 5400 50  0001 C CNN
 F 3 "~" H 3300 5550 50  0001 C CNN
 	1    3300 5550
@@
 F 0 "SW1" V 3604 5698 50  0000 L CNN
 F 1 "PWR_RES" V 3695 5698 50  0000 L CNN
-F 2 "" H 3650 5750 50  0001 C CNN
+F 2 "Button_Switch_THT:SW_PUSH_6mm" H 3650 5750 50  0001 C CNN
 F 3 "~" H 3650 5750 50  0001 C CNN
 	1    3650 5550
@@
 F 0 "C1" H 2868 7246 50  0000 L CNN
 F 1 ".22uF" H 2868 7155 50  0000 L CNN
-F 2 "" H 2788 7050 50  0001 C CNN
+F 2 "Capacitor_THT:CP_Radial_D5.0mm_P2.50mm" H 2788 7050 50  0001 C CNN
 F 3 "~" H 2750 7200 50  0001 C CNN
 	1    2750 7200
@@
 F 0 "C3" H 4018 7246 50  0000 L CNN
 F 1 ".1uF" H 4018 7155 50  0000 L CNN
-F 2 "" H 3938 7050 50  0001 C CNN
+F 2 "Capacitor_THT:CP_Radial_D5.0mm_P2.50mm" H 3938 7050 50  0001 C CNN
 F 3 "~" H 3900 7200 50  0001 C CNN
 	1    3900 7200
@@
 F 0 "C5" H 4600 5850 50  0000 L CNN
 F 1 ".01uF" H 4550 5700 50  0000 L CNN
-F 2 "" H 4838 5650 50  0001 C CNN
+F 2 "Capacitor_THT:C_Disc_D7.5mm_W5.0mm_P7.50mm" H 4838 5650 50  0001 C CNN
 F 3 "~" H 4800 5800 50  0001 C CNN
 	1    4800 5800
@@
 F 0 "C6" H 6518 6046 50  0000 L CNN
 F 1 "10uF" H 6518 5955 50  0000 L CNN
-F 2 "" H 6438 5850 50  0001 C CNN
+F 2 "Capacitor_THT:CP_Radial_D5.0mm_P2.50mm" H 6438 5850 50  0001 C CNN
 F 3 "~" H 6400 6000 50  0001 C CNN
 	1    6400 6000
@@
 F 0 "R1" H 6470 5446 50  0000 L CNN
 F 1 "10k" H 6470 5355 50  0000 L CNN
-F 2 "" V 6330 5400 50  0001 C CNN
+F 2 "Resistor_THT:R_Axial_DIN0207_L6.3mm_D2.5mm_P7.62mm_Horizontal" V 6330 5400 50  0001 C CNN
 F 3 "~" H 6400 5400 50  0001 C CNN
 	1    6400 5400
@@
 F 0 "R2" H 6330 5654 50  0000 R CNN
 F 1 "10k" H 6330 5745 50  0000 R CNN
-F 2 "" V 6330 5700 50  0001 C CNN
+F 2 "Resistor_THT:R_Axial_DIN0207_L6.3mm_D2.5mm_P7.62mm_Horizontal" V 6330 5700 50  0001 C CNN
 F 3 "~" H 6400 5700 50  0001 C CNN
 	1    6400 5700
@@
 F 0 "C4" H 5100 7250 50  0000 L CNN
 F 1 ".1uF" H 5200 7250 50  0000 L CNN
-F 2 "" H 5238 7000 50  0001 C CNN
+F 2 "Capacitor_THT:C_Disc_D4.3mm_W1.9mm_P5.00mm" H 5238 7000 50  0001 C CNN
 F 3 "~" H 5200 7150 50  0001 C CNN
 	1    5200 7150
@@
 F 0 "C7" H 5400 7250 50  0000 L CNN
 F 1 ".1uF" H 5500 7250 50  0000 L CNN
-F 2 "" H 5538 7000 50  0001 C CNN
+F 2 "Capacitor_THT:C_Disc_D4.3mm_W1.9mm_P5.00mm" H 5538 7000 50  0001 C CNN
 F 3 "~" H 5500 7150 50  0001 C CNN
 	1    5500 7150
@@
 F 0 "C8" H 5700 7250 50  0000 L CNN
 F 1 ".1uF" H 5800 7250 50  0000 L CNN
-F 2 "" H 5838 7000 50  0001 C CNN
+F 2 "Capacitor_THT:C_Disc_D4.3mm_W1.9mm_P5.00mm" H 5838 7000 50  0001 C CNN
 F 3 "~" H 5800 7150 50  0001 C CNN
 	1    5800 7150
@@
 F 0 "C9" H 6000 7250 50  0000 L CNN
 F 1 ".1uF" H 6100 7250 50  0000 L CNN
-F 2 "" H 6138 7000 50  0001 C CNN
+F 2 "Capacitor_THT:C_Disc_D4.3mm_W1.9mm_P5.00mm" H 6138 7000 50  0001 C CNN
 F 3 "~" H 6100 7150 50  0001 C CNN
 	1    6100 7150
